File: elec/bucket.sch (EAGLE design)
At the start: 4 parts, among them U1 PCF85263ATT/AJ-SO8

Commit message: major progress on circuit design
Parts:
- removed BAT1: BATT-COIN-KEYSTONE-3001, bucket:BATT-COIN-KEYSTONE-3001
- removed U1: PCF85263ATT/AJ-SO8, bucket:PCF85263ATT/AJ-SO8
- added C1: 47uF, bucket:CAP_POLD
- added C2, C9: 100nF, bucket:CAP0603-CAP
- added C3, C4: 2u2, bucket:CAP0603-CAP
- added C5, C6, C7, C8: 1uF, bucket:CAP0603-CAP
- added D1, D2: (no value), bucket:DIODESMB
- added D3, D4: 2V4, bucket:DIODE-ZENER-SOD323
- added IC1: PSU-OKRT6, bucket:PSU-OKRT6
- added JP1, JP2: (no value), bucket:M02POLAR
- added LS1: CT-1205C-SMT, bucket:CT-1205C-SMT
- added Q1: MOSFET-NCHAN, bucket:MOSFET-NCHANNELSMD
- added R1, R13, R14, R15, R16, R17, R18, R19, R2, R5, R7: 4K7, bucket:RESISTOR0603-RES
- added R10, R11, R12, R8, R9: 0R, bucket:RESISTOR0603-RES
- added R3: 267R, bucket:RESISTOR0603-RES
- added R4, R6: 15K, bucket:RESISTOR0603-RES
- added S1, S2, S3, S4, S5: (no value), bucket:TAC_SWITCHPTH
- added U2: MAX1037EKA, bucket:MAX1037EKA
- RPI1: value RASPBERRY_PI_3_MODEL_B+ -> RASPBERRY PI
Connections:
- new net 3.3V: C2.1, C9.2, OLED1.VBAT, OLED1.VDD, R1.2, R11.1, R15.2, R16.2, R17.2, R18.2, R19.2, R2.2, RPI1.3V3, U2.VDD
- new net 5V: C1.+, IC1.VOUT, LS1.1, RPI1.5V0
- new net ADC-BAT-1: C7.2, D3.C, R6.2, R7.1, U2.AIN0
- new net ADC-BAT-2: C8.1, D4.C, R4.1, R5.2, U2.AIN1
- new net BTN1: R15.1, RPI1.GPIO19, S1.1, S1.2
- new net BTN2: R16.1, RPI1.GPIO16, S2.1, S2.2
- new net BTN3: R17.1, RPI1.GPIO26, S3.1, S3.2
- new net BTN4: R18.1, RPI1.GPIO20, S4.1, S4.2
- new net BTN5: R19.1, RPI1.GPIO21, S5.1, S5.2
- new net BUZZER: R13.2, R14.1, RPI1.GPIO13
- new net GND: C1.-, C2.2, C3.2, C4.2, C7.1, C8.2, C9.1, D3.A, D4.A, IC1.GND, JP1.1, JP2.1, OLED1.VSS, Q1.S, R12.1, R14.2, R3.1, R5.1, R7.2, R8.1, RPI1.GND, RPI1.SHIELD, S1.3, S1.4, S2.3, S2.4, S3.3, S3.4, S4.3, S4.4, S5.3, S5.4, U2.GND
- new net N$1: D2.A, JP2.2, R4.2
- new net N$10: OLED1.SDA/MOSI, R10.2
- new net N$11: OLED1.BS1, R11.2
- new net N$12: OLED1.BS0, R12.2
- new net N$13: C4.1, OLED1.VCOMH
- new net N$14: C3.1, OLED1.VCC
- new net N$16: C5.2, OLED1.C1N
- new net N$17: C5.1, OLED1.C1P
- new net N$18: C6.1, OLED1.C2P
- new net N$19: C6.2, OLED1.C2N
- new net N$2: D1.A, JP1.2, R6.1
- new net N$3: D1.C, D2.C, IC1.VIN
- new net N$4: IC1.TRIM, R3.2
- new net N$5: Q1.G, R13.1
- new net N$6: LS1.2, Q1.D
- new net N$7: OLED1.D/!C, R8.2
- new net N$9: OLED1.SDA/MISO, R9.2
- new net OLED-CS: OLED1.!CS, RPI1.GPIO27/GPIO_GEN2
- new net OLED-RST: OLED1.!RES, RPI1.GPIO17/GPIO_GEN0
- new net SCL: OLED1.SCLK, R2.1, RPI1.GPIO3/SCL1, U2.SCL
- new net SDA: R1.1, R10.1, R9.1, RPI1.GPIO2/SDA1, U2.SDA
Other:
- note added: "8.4V battery inputs"
- note added: "divider, 8.5V to 2.028V"
- note added: "set for about 5V"
- moved on the sheet: OLED1, RPI1

Commit message: circuit first rev finished and gerbers sent to manufacture
Parts:
- removed JP2: (no value), bucket:M02POLAR
- JP1: device bucket:M02POLAR -> bucket:M04-AMPMODUMTE-TH-ANG
- renumbered S1 to SW1, S2 to SW2, S3 to SW3, S4 to SW4, S5 to SW5
Connections:
- net GND: now also JP1.4; no longer JP2.1
- net N$1: now also JP1.3; no longer JP2.2

Commit message: PCB v2
Parts:
- removed C4: 2u2, bucket:CAP0603-CAP
- removed C5, C6, C7, C8: 1uF, bucket:CAP0603-CAP
- removed C9: 100nF, bucket:CAP0603-CAP
- removed D1, D2: (no value), bucket:DIODESMB
- removed D3, D4: 2V4, bucket:DIODE-ZENER-SOD323
- removed IC1: PSU-OKRT6, bucket:PSU-OKRT6
- removed JP1: (no value), bucket:M04-AMPMODUMTE-TH-ANG
- removed OLED1: EA-OLEDS102-6, bucket:EA-OLEDS102-6
- removed U2: MAX1037EKA, bucket:MAX1037EKA
- added R20: 0R, bucket:RESISTOR0603-RES
- added SW6: (no value), bucket:TAC_SWITCHPTH
- added U$1: OLED-PANEL-1.54IN, bucket:OLED-PANEL-1.54IN
- added U1: OLED-CONN, bucket:OLED-CONN
- C1: value 47uF -> 100nF; device bucket:CAP_POLD -> bucket:CAP0603-CAP
- C3: value 2u2 -> 4u7
- R3: value 267R -> 910K
- R4, R6: value 15K -> 0R
- R5, R7: value 4K7 -> 0R
- renumbered LS1 to BUZZER
Connections:
- removed net ADC-BAT-1: C7.2, D3.C, R6.2, R7.1, U2.AIN0
- removed net ADC-BAT-2: C8.1, D4.C, R4.1, R5.2, U2.AIN1
- removed net N$16: C5.2, OLED1.C1N
- removed net N$17: C5.1, OLED1.C1P
- removed net N$18: C6.1, OLED1.C2P
- removed net N$19: C6.2, OLED1.C2N
- new net N$8: R7.1, U1.RW
- net 3.3V: now also C1.1, R4.2, U1.VCC, U1.VDD; no longer C9.2, OLED1.VBAT, OLED1.VDD, R11.1, U2.VDD
- net 5V: no longer C1.+, IC1.VOUT
- net BTN1: now also RPI1.GPIO18/GPIO_GEN1; no longer RPI1.GPIO19
- net BTN2: now also RPI1.GPIO22/GPIO_GEN3; no longer RPI1.GPIO16
- net BTN3: now also RPI1.GPIO23/GPIO_GEN4; no longer RPI1.GPIO26
- net BTN4: now also RPI1.GPIO10/SPI_MOSI; no longer RPI1.GPIO20
- net BTN5: now also RPI1.GPIO24/GPIO_GEN5; no longer RPI1.GPIO21
- net BUZZER: now also RPI1.GPIO26; no longer RPI1.GPIO13
- net GND: now also C1.2, R3.2, R5.2, R6.2, R8.2, SW6.3, SW6.4, U1.MNT1, U1.MNT2, U1.NC-GND-1, U1.NC-GND-2, U1.VLSS, U1.VSS; no longer C1.-, C4.2, C7.1, C8.2, C9.1, D3.A, D4.A, IC1.GND, JP1.1, JP1.4, OLED1.VSS, R12.1, R3.1, R5.1, R8.1, U2.GND
- net N$1: now also C3.1, U1.VCOMH; no longer D2.A, JP1.3, R4.2
- net N$10: now also R9.1, U1.CS; no longer OLED1.SDA/MOSI, R10.2
- net N$11: now also R10.2, U1.RES; no longer OLED1.BS1, R11.2
- net N$12: now also R11.2, U1.D0/SCL; no longer OLED1.BS0, R12.2
- net N$13: now also R12.2, U1.D1/SDA; no longer C4.1, OLED1.VCOMH
- net N$14: now also R20.2, U1.D2/SDA; no longer C3.1, OLED1.VCC
- net N$2: now also R3.1, U1.IREF; no longer D1.A, JP1.2, R6.1
- net N$3: now also R4.1, U1.BS1; no longer D1.C, D2.C, IC1.VIN
- net N$4: now also R5.1, U1.BS2; no longer IC1.TRIM, R3.2
- net N$7: now also R6.1, U1.SA0; no longer OLED1.D/!C, R8.2
- net N$9: now also R8.1, U1.ERD; no longer OLED1.SDA/MISO, R9.2
- net OLED-CS: now also R9.2, RPI1.GPIO17/GPIO_GEN0; no longer OLED1.!CS, RPI1.GPIO27/GPIO_GEN2
- net OLED-RST: now also R10.1, RPI1.GPIO27/GPIO_GEN2; no longer OLED1.!RES, RPI1.GPIO17/GPIO_GEN0
- net SCL: now also R11.1; no longer OLED1.SCLK, U2.SCL
- net SDA: now also R12.1, R20.1; no longer R10.1, R9.1, U2.SDA
Other:
- note removed: "8.4V battery inputs"
- note removed: "divider, 8.5V to 2.028V"
- note removed: "set for about 5V"
- moved on the sheet: C2, C3, R10, R11, R12, R3, R4, R5, R6, R7, R8, R9
